File: Cabina.kicad_pcb (KiCad board)
At the start: 4 copper layers, 99.5 x 92.4 mm, 104 parts, among them J100 VCC INPUT, J101 SWITCH ON/OFF, J103 FAN VOLTAGE, J200 LIGHT SWITCH & LED STRIP, J201 LIGHT SWITCH & LED STRIP, J202 LIGHT SWITCH & LED STRIP, J203 LED STRIP, J300 Serial Wire Debug, J301 CAN_ID_CONFIG, J302 CAN_INPUT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

Commit message: change board stackup
Parts:
- L101: footprint Jose_:SMD_12.3X12.3mm -> Inductor_SMD:SMD_12.3X12.3mm
- moved G*** 2.78 mm to (150.1, 78.6)
Routing:
- net GND: vias 361 -> 347

Commit message: version validada
Parts:
- D200, D204, D208, D213: footprint Diode_SMD:D_SOD-128 -> Diode_SMD:Nexperia_CFP3_SOD-123W
- J101: footprint Connector_PinHeader_2.54mm:PinHeader_1x02_P2.54mm_Vertical -> B2B-XH-A:JST_B2B-XH-A_LF__SN_
- moved TP100 3.05 mm to (116.4, 41.6)
- moved TP101 2.92 mm to (120.4, 41.6)
- moved J101 2.33 mm to (128.2, 41.5), turned to 0 degrees
Routing:
- net /POWER/V_INPUT: track 34.0 -> 36.7 mm
- net GND: track 56.2 -> 58.2 mm, vias 347 -> 344
- net Net-(D213-A): track 5.18 -> 6.03 mm
- net 24V_HEADBOARD: track 37.2 -> 38.0 mm
- net 24V_CEILING: track 41.0 -> 41.8 mm
- net /RELAYS/24v_headboard: track 8.16 -> 8.96 mm
- net /RELAYS/24v_ceiling: track 8.41 -> 9.21 mm
- net /RELAYS/24V_SIGN: track 15.5 -> 16.3 mm
- net 24V_TABLE: track 38.3 -> 39.1 mm
- net /RELAYS/24v_table: track 6.73 -> 7.53 mm
