File: RELAYS.kicad_sch (KiCad schematic)
At the start: 40 parts, among them J200 LIGHT SWITCH & LED STRIP, J201 LIGHT SWITCH & LED STRIP, J202 LIGHT SWITCH & LED STRIP, J203 LED STRIP, K200 RELAY_HEADBOARD, K201 RELAY_TABLE, K202 RELAY_CEILING, K203 RELAY_SIGN, Q200 MMBT3904, Q201 MMBT3904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

Commit message: change board stackup
Parts:
- D200, D204, D208, D213: LCSC (none) -> C513108
Changed lines of the file:
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@@
+      (effects (font (size 1.27 1.27)) hide)
+    )
+    (property "LCSC" " C513108" (at 71.628 41.275 0)
       (effects (font (size 1.27 1.27)) hide)
     )
@@
       (effects (font (size 1.27 1.27)) hide)
     )
+    (property "LCSC" " C513108" (at 72.644 118.11 0)
+      (effects (font (size 1.27 1.27)) hide)
+    )
     (pin "1")
     (pin "2")
@@
       (effects (font (size 1.27 1.27)) hide)
     )
+    (property "LCSC" " C513108" (at 198.374 116.713 0)
+      (effects (font (size 1.27 1.27)) hide)
+    )
     (pin "1")
     (pin "2")
@@
       (effects (font (size 1.27 1.27)) hide)
     )
+    (property "LCSC" " C513108" (at 211.582 29.21 0)
+      (effects (font (size 1.27 1.27)) hide)
+    )

Commit message: version validada
Parts:
- D200, D204, D208, D213: footprint Diode_SMD:D_SOD-128 -> Diode_SMD:Nexperia_CFP3_SOD-123W; LCSC C513108 -> C552879
Changed lines of the file:
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@@
       (effects (font (size 1.27 1.27)))
     )
-    (property "Footprint" "Diode_SMD:D_SOD-128" (at 71.628 45.72 0)
+    (property "Footprint" "Diode_SMD:Nexperia_CFP3_SOD-123W" (at 71.628 45.72 0)
       (effects (font (size 1.27 1.27)) hide)
     )
@@
       (effects (font (size 1.27 1.27)) hide)
     )
-    (property "LCSC" " C513108" (at 71.628 41.275 0)
+    (property "LCSC" "C552879" (at 71.628 41.275 0)
       (effects (font (size 1.27 1.27)) hide)
     )
@@
       (effects (font (size 1.27 1.27)))
     )
-    (property "Footprint" "Diode_SMD:D_SOD-128" (at 72.644 122.555 0)
+    (property "Footprint" "Diode_SMD:Nexperia_CFP3_SOD-123W" (at 72.644 122.555 0)
       (effects (font (size 1.27 1.27)) hide)
     )
@@
       (effects (font (size 1.27 1.27)) hide)
     )
-    (property "LCSC" " C513108" (at 72.644 118.11 0)
+    (property "LCSC" "C552879" (at 72.644 118.11 0)
       (effects (font (size 1.27 1.27)) hide)
     )
@@
       (effects (font (size 1.27 1.27)))
     )
-    (property "Footprint" "Diode_SMD:D_SOD-128" (at 198.374 121.158 0)
+    (property "Footprint" "Diode_SMD:Nexperia_CFP3_SOD-123W" (at 198.374 121.158 0)
       (effects (font (size 1.27 1.27)) hide)
     )
@@
       (effects (font (size 1.27 1.27)) hide)
     )
-    (property "LCSC" " C513108" (at 198.374 116.713 0)
+    (property "LCSC" "C552879" (at 198.374 116.713 0)
       (effects (font (size 1.27 1.27)) hide)
     )
@@
       (effects (font (size 1.27 1.27)))
     )
-    (property "Footprint" "Diode_SMD:D_SOD-128" (at 211.582 33.655 0)
+    (property "Footprint" "Diode_SMD:Nexperia_CFP3_SOD-123W" (at 211.582 33.655 0)
       (effects (font (size 1.27 1.27)) hide)
     )
@@
       (effects (font (size 1.27 1.27)) hide)
     )
-    (property "LCSC" " C513108" (at 211.582 29.21 0)
-      (effects (font (size 1.27 1.27)) hide)
-    )
+    (property "LCSC" "C552879" (at 211.582 29.21 0)
+      (effects (font (size 1.27 1.27)) hide)
+    )
