File: power.kicad_sch (KiCad schematic)
At the start: 22 parts, among them J100 VCC INPUT, J101 SWITCH ON/OFF, J103 FAN VOLTAGE, Q100 WST4045, U100 LM2596S-5, U101 AMS1117-3.3

Commit message: version validada
Parts:
- D103: LCSC C72043 -> C72038
- J101: footprint Connector_PinHeader_2.54mm:PinHeader_1x02_P2.54mm_Vertical -> B2B-XH-A:JST_B2B-XH-A_LF__SN_
Changed lines of the file:
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@@
       (effects (font (size 1.27 1.27)) hide)
     )
-    (property "LCSC" "C72043" (at 209.042 77.343 0)
+    (property "LCSC" "C72038" (at 209.042 77.343 0)
       (effects (font (size 1.27 1.27)) hide)
     )
@@
       (effects (font (size 1.27 1.27)) (justify right))
     )
-    (property "Footprint" "Connector_PinHeader_2.54mm:PinHeader_1x02_P2.54mm_Vertical" (at 78.74 64.135 0)
+    (property "Footprint" "B2B-XH-A:JST_B2B-XH-A_LF__SN_" (at 78.74 64.135 0)
       (effects (font (size 1.27 1.27)) hide)
     )
